File: EncKiboard_V2.sch (KiCad schematic (older format))
At the start: 44 parts, among them IC1 4094D, IC2 4094D, SW1 Rotary_Encoder_Switch, U0 ProMicro, U1 CherryMX_LED, U10 CherryMX_LED, U11 CherryMX_LED, U12 CherryMX_LED, U2 CherryMX_LED, U3 CherryMX_LED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

Commit message: Edit wrong diode position
Parts:
- removed D10, D11, D12, D13, D14, D3, D4, D5, D6, D7, D8, D9: DIODE, Diode_SMD:D_MELF_Handsoldering, symbol pspice:DIODE
- added D10, D11, D12, D13, D14, D3, D4, D5, D6, D7, D8, D9: 1N4148_SMD, Diode_SMD:D_MELF_Handsoldering, symbol Diode:SM4004
Connections:
- wire segments 158 -> 170
